Commit message: finished joints

File: body.urdf (robot description, URDF)
Before this commit: robot robot, 4 links, 3 joints
Links:
- removed link Link0
- removed link Link1
- removed link Link2
- removed link Link3
- added link BackLeg, mass 1; collision box size=1 1 1; visual box size=1 1 1
- added link FrontLeg, mass 1; collision box size=1 1 1; visual box size=1 1 1
- added link Torso, mass 1; collision box size=1 1 1; visual box size=1 1 1
Joints:
- removed joint Link0_Link1
- removed joint Link1_Link2
- removed joint Link2_Link3
- added joint BackLeg_FrontLeg: type revolute, parent BackLeg, child FrontLeg, origin xyz=0 1 0 rpy=0 0 0, axis 0 1 0, limit lower=-3.14159 upper=3.14159 effort=0.0 velocity=0.0
- added joint Torso_BackLeg: type revolute, parent Torso, child BackLeg, origin xyz=0 0.5 1 rpy=0 0 0, axis 0 1 0, limit lower=-3.14159 upper=3.14159 effort=0.0 velocity=0.0

Commit message: fixed the shape

File: body.urdf (robot description, URDF)
Before this commit: robot robot, 3 links, 2 joints
Joints:
- joint BackLeg_FrontLeg: origin xyz=0 1 0 rpy=0 0 0 -> xyz=1 0 0 rpy=0 0 0
- joint Torso_BackLeg: origin xyz=0 0.5 1 rpy=0 0 0 -> xyz=0.5 0 1 rpy=0 0 0
